File: Hardware/GMCounter.sch (KiCad schematic (older format))
At the start: 18 parts, among them Q1 IRF820, SW1 ON_SWITCH, SW2 RST_CNT, U1 TPS6650, U2 MSP430G2553, U3 TPS6533, U4 LM358, U5 OPA2350, Y1 Crystal

Commit message: Started PCB design over again
Parts:
- removed C3: GEIGER_MUELLER, symbol GEIGER_MUELLER
- removed U1: TPS6650, ~, symbol TPS6xxx
- removed U2: MSP430G2553, symbol MSP430G2553
- removed U3: TPS6533, ~, symbol TPS6xxx
- removed U5: OPA2350, symbol OPA2350
- added DS?: LCD16X2, WC1602A, symbol LCD16X2
- added U?: TPS76650, symbol TPS76650
- added U?: TPS76533, symbol TPS76533
- added U?: MSP430G2253IN20, 20N, symbol MSP430G2253IN20
- D1, D2: footprint LEDs:LED-0805 -> LEDs:LED-1206
Changed lines of the file:
@@
 EESchema Schematic File Version 2
-LIBS:CustomDevices
 LIBS:power
 LIBS:device
@@
 LIBS:contrib
 LIBS:valves
-LIBS:Components
+LIBS:msp430
+LIBS:powerint
+LIBS:GM_components
 LIBS:GMCounter-cache
 EELAYER 25 0
@@
 F 0 "D2" H 4350 1500 50  0000 C CNN
 F 1 "LED" H 4350 1300 50  0000 C CNN
-F 2 "LEDs:LED-0805" H 4400 1200 60  0000 C CNN
+F 2 "LEDs:LED-1206" H 4400 1200 60  0000 C CNN
 F 3 "" H 4350 1400 60  0000 C CNN
 	1    4350 1400
@@
 F 3 "" H 1950 4850 60  0000 C CNN
 	1    1950 4850
-	1    0    0    -1
-$EndComp
-$Comp
-L TPS6xxx U1
-U 1 1 5602DE82
-P 2350 3750
-F 0 "U1" H 2350 3400 60  0000 C CNN
-F 1 "TPS6650" H 2350 4150 60  0000 C CNN
-F 2 "~" H 2400 3300 60  0000 C CNN
-F 3 "" H 2350 3750 60  0000 C CNN
-	1    2350 3750
-	1    0    0    -1
-$EndComp
-$Comp
-L TPS6xxx U3
-U 1 1 5602E177
-P 4350 3950
-F 0 "U3" H 4350 3600 60  0000 C CNN
-F 1 "TPS6533" H 4350 4350 60  0000 C CNN
-F 2 "~" H 4400 3500 60  0000 C CNN
-F 3 "" H 4350 3950 60  0000 C CNN
-	1    4350 3950
-	1    0    0    -1
-$EndComp
-$Comp
-L MSP430G2553 U2
-U 1 1 56030706
-P 3050 5300
-F 0 "U2" H 3050 4750 60  0000 C CNN
-F 1 "MSP430G2553" H 3050 5900 60  0000 C CNN
-F 2 "" H 3100 5400 60  0000 C CNN
-F 3 "" H 3100 5400 60  0000 C CNN
-	1    3050 5300
-	1    0    0    -1
-$EndComp
-$Comp
-L GEIGER_MUELLER C3
-U 1 1 56030E95
-P 5100 5300
-F 0 "C3" H 5100 5250 60  0000 C CNN
-F 1 "GEIGER_MUELLER" H 5100 5400 60  0000 C CNN
-F 2 "" H 5100 5300 60  0000 C CNN
-F 3 "" H 5100 5300 60  0000 C CNN
-	1    5100 5300
 	1    0    0    -1
 $EndComp
@@
 	-1   0    0    1
 $EndComp
-$Comp
-L OPA2350 U5
-U 1 1 560338AB
-P 8550 1550
-F 0 "U5" H 8500 1750 60  0000 L CNN
-F 1 "OPA2350" H 8500 1300 60  0000 L CNN
-F 2 "" H 8550 1550 60  0000 C CNN
-F 3 "" H 8550 1550 60  0000 C CNN
-	1    8550 1550
-	1    0    0    -1
-$EndComp
-$Comp
-L OPA2350 U5
-U 2 1 56033911
-P 8550 2550
-F 0 "U5" H 8500 2750 60  0000 L CNN
-F 1 "OPA2350" H 8500 2300 60  0000 L CNN
-F 2 "" H 8550 2550 60  0000 C CNN
-F 3 "" H 8550 2550 60  0000 C CNN
-	2    8550 2550
-	1    0    0    -1
-$EndComp
 Text Label 1700 5150 0    60   ~ 0
 AUDIO_OUT
@@
 F 0 "D1" H 1400 3400 50  0000 C CNN
 F 1 "LED" H 1400 3200 50  0000 C CNN
-F 2 "LEDs:LED-0805" H 1450 3100 60  0000 C CNN
+F 2 "LEDs:LED-1206" H 1450 3100 60  0000 C CNN
 F 3 "" H 1400 3300 60  0000 C CNN
 	1    1400 3300
@@
 	2550 4600 2550 4850
 Connection ~ 2550 4850
+$Comp
+L MSP430G2253IN20 U?
+U 1 1 5627FC8A
+P 3450 6750
+F 0 "U?" H 1950 7350 40  0000 C CNN
+F 1 "MSP430G2253IN20" H 4700 6200 40  0000 C CNN
+F 2 "20N" H 2000 6200 35  0000 C CIN
+F 3 "" H 3400 6750 60  0000 C CNN
+	1    3450 6750
+	1    0    0    -1
+$EndComp
+$Comp
+L LCD16X2 DS?
+U 1 1 56280145
+P 7750 5550
+F 0 "DS?" H 6950 5950 40  0000 C CNN
+F 1 "LCD16X2" H 8450 5950 40  0000 C CNN
+F 2 "WC1602A" H 7750 5500 35  0000 C CIN
+F 3 "" H 7750 5550 60  0000 C CNN
+	1    7750 5550
+	1    0    0    -1
+$EndComp
+$Comp
+L TPS76650 U?
+U 1 1 5627F562
+P 2350 3850
+F 0 "U?" H 2350 3550 60  0000 C CNN
+F 1 "TPS76650" H 2350 4500 60  0000 C CNN
+F 2 "" H 2350 3850 60  0000 C CNN
+F 3 "" H 2350 3850 60  0000 C CNN
+	1    2350 3850
+	1    0    0    -1
+$EndComp
+$Comp
+L TPS76533 U?
+U 1 1 5627F93E
+P 4350 3900
+F 0 "U?" H 4350 3600 60  0000 C CNN
+F 1 "TPS76533" H 4350 4550 60  0000 C CNN
+F 2 "" H 4350 3900 60  0000 C CNN
+F 3 "" H 4350 3900 60  0000 C CNN
+	1    4350 3900
+	1    0    0    -1
+$EndComp
 $EndSCHEMATC

Commit message: Working on schematics
Parts:
- removed C1: C, symbol C
- removed C2: CP, symbol CP
- removed Q1: IRF820, symbol Q_NMOS_GDS
- removed R2: R, symbol R
- added C?: 150n, symbol C
- added C? (x2): 4u7, symbol CP
- added C? (x2): 100n, symbol C
- added D?: 1N4007, symbol D
- added D?: YELLOW_LED, LEDs:LED-1206, symbol LED
- added Q?: 2N3904, symbol Q_NPN_EBC
- added Q?: 2N3906, symbol Q_PNP_EBC
- added Q?: IRF820, symbol Q_NMOS_GDS
- added R?: 470, symbol R
- added R?: 560, symbol R
- added R?: 110, symbol R
- added R?: 4M7, symbol R
- added SW?: USR_BTN, symbol SW_PUSH
- D2: value LED -> BLUE_LED
- R1: value 10k -> 6k8
Connections:
- net labels added: HV_OUT, LCD_D4, LCD_D5, LCD_D6, LCD_D7, LCD_EN, LCD_LD, LCD_RS, PUSH_BTN, USER_BTN
- wire segments 53 -> 119
Other:
- moved on the sheet: DS?, L1, SW2, Y1

Commit message: First complete schematic commit
Parts:
- added C1: 22p, symbol C
- added C6: 1n, symbol C
- added D2: 1N4148, symbol D
- added P1: GM_CONN, symbol CONN_01X02
- added P2: BATT_CONN, symbol CONN_01X02
- added P3: ICSP, symbol CONN_01X04
- added Q4: 2N3904, symbol Q_NPN_EBC
- added R10, R11: 1k, symbol R
- added R12: 4k7, symbol R
- added R2: 220, symbol R
- added R3: 51k, symbol R
- added R4: 27k, symbol R
- added R5: 47k, symbol R
- added R6: 330k, symbol R
- added U2: OPA2350, symbol OPA2350
- D1: value LED -> RED_LED
- SP1: value SPEAKER -> BUZZER
- Y1: value Crystal -> 32.768 kHz
- gave numbers to parts that had none: 19
- renumbered D2 to D4, U4 to U5
Connections:
- net labels added: BATT_INPUT, GM_A+, GM_K-, LCD_LD_B, LED_CNT, LED_WRNG, RST, TEST
- wire segments 119 -> 190
Other:
- note added: "DETECTOR\nSTAGE"
- note added: "HV STAGE"
- note added: "MICROCONTROLLER"
- note added: "POWER SUPPLY &\nVOLTAGE REGULATION"
- note added: "USER INTERFACE"
- note added: "uC ICSP"
- moved on the sheet: C2, C3, C4, C5, R1, SP1, SW1, SW2, SW3, U1, U3, U4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
