File: Hardware/GMCounter.kicad_pcb (KiCad board)
At the start: 2 copper layers, 99.1 x 94 mm, 58 parts, among them P1 GM_CONN, P10 TP, P11 TP, P12 TP, P13 TP, P14 TP, P2 TP, P3 TP, P4 TP, P5 BATT_CONN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

Commit message: Preliminary PCB design
Parts:
- C1, R10, R11, R12, R2, R3, R4, R5, R7, R9, U2: moved to B.Cu
- moved DS1 122.7 mm to (71.9, 129.2)
- moved Q3 110.1 mm to (128.6, 53.5), turned to 180 degrees
- moved Y1 90.4 mm to (71.5, 108.4)
- moved U3 88.9 mm to (74.2, 120.4), turned to 90 degrees
- moved L1 88.4 mm to (143.3, 63.1)
- moved P8 85.4 mm to (84.4, 106.7), turned to 270 degrees
- moved D2 85.0 mm to (138.9, 113.4), turned to 180 degrees
- moved R8 84.9 mm to (133.3, 117.7), turned to 0 degrees
- moved D5 83.5 mm to (142.7, 85.6), turned to 180 degrees
- moved P10 82.3 mm to (129.2, 104.8), turned to 180 degrees
- moved R3 79.7 mm to (104.0, 57.6), turned to 90 degrees
- moved U5 78.1 mm to (135.1, 107.6)
- moved SP1 76.4 mm to (121.5, 107.4), turned to 270 degrees
- moved C7 73.9 mm to (126.0, 85.6), turned to 180 degrees
- moved R2 69.7 mm to (105.4, 61.5), turned to 180 degrees
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Routing:
- net GND: track 0.00 -> 394.4 mm, vias 0 -> 1
- net +5V: track 0.00 -> 272.4 mm
- net +3V3: track 0.00 -> 158.8 mm, vias 0 -> 4
- net /FREQ_OUT: track 0.00 -> 90.9 mm, vias 0 -> 4
- net Net-(D5-Pad1): track 0.00 -> 60.8 mm
- net /GM_A+: track 0.00 -> 59.6 mm
- net /AUDIO_OUT: track 0.00 -> 49.2 mm
- net /PULSE_IN: track 0.00 -> 48.9 mm, vias 0 -> 3
- net /BATT_INPUT: track 0.00 -> 32.0 mm
- net +BATT: track 0.00 -> 29.6 mm, vias 0 -> 2
- net /PUSH_BTN: track 0.00 -> 29.5 mm
- net /LED_CNT: track 0.00 -> 28.6 mm, vias 0 -> 1
- net /LCD_LD_B: track 0.00 -> 28.2 mm
- net Net-(C1-Pad1): track 0.00 -> 23.4 mm, vias 0 -> 1
- net Net-(P11-Pad1): track 0.00 -> 21.3 mm
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- added copper zone on B.Cu, net GND
- added copper zone on F.Cu, net GND
Other:
- board text added: "3v3"
- board text added: "Contador GM"
- board text added: "D"
- board text added: "Diseño Ing. Iván Morales"
- board text added: "ECFM"
- board text added: "G"
- board text added: "GND"
- board text added: "Guatemala, Enero 2016"
- board text added: "Laboratorio de Instrumentación"
- board text added: "RST"
- board text added: "S"
- board text added: "TST"
- board text added: "USAC"

Commit message: Updated preliminary PCB design with ECFM logo
Parts:
- added ?: , LOGO, F.Cu at (63.5, 52.1)

Commit message: First calibration hardware design commit
Other:
- board text added: "Monterroso, Andrés Morales, Iván Urizar, Silvio"
- board text removed: "Diseño Ing. Iván Morales"
Changed lines of the file:
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@@
     (links 118)
     (no_connects 0)
-    (area 36.894501 42.799 152.908001 163.033005)
+    (area 53.734499 42.812499 152.894501 136.892501)
     (thickness 1.6)
     (drawings 20)
@@
   (page A4)
   (layers
-    (0 F.Cu signal hide)
+    (0 F.Cu signal)
     (31 B.Cu signal)
     (32 B.Adhes user hide)
@@
     (effects (font (size 1.5 1.5) (thickness 0.3)))
   )
-  (gr_text "Diseño\nIng. Iván Morales" (at 83.058 58.039) (layer B.SilkS)
-    (effects (font (size 2 2) (thickness 0.4)) (justify mirror))
+  (gr_text "Monterroso, Andrés\nMorales, Iván\nUrizar, Silvio" (at 79.375 54.229) (layer B.SilkS)
+    (effects (font (size 1.5 1.5) (thickness 0.3)) (justify mirror))
   )
   (gr_text USAC (at 82.931 60.96) (layer F.Mask)

Commit message: PCB Release Candidate
Parts:
- removed D3: YELLOW_LED, LEDs:LED-1206
- removed R13: 1k, Resistors_SMD:R_0805_HandSoldering
- added C8: 100n, Capacitors_SMD:C_0805_HandSoldering, F.Cu at (135.4, 112.9)
- added RV1: POT, Potentiometers:Potentiometer_Alps-RK16-single_largePads, F.Cu at (146.6, 92.1)
- P14: footprint Measurement_Points:Measurement_Point_Round-TH_Small -> Pin_Headers:Pin_Header_Straight_1x01
- moved P4 13.2 mm to (57.5, 80.0)
- moved R8 5.63 mm to (135.9, 122.7)
- moved D2 5.32 mm to (137.3, 118.5)
- moved ? 1.85 mm to (65.3, 51.6)
- moved P14 1.49 mm to (114.2, 95.1)
Connections:
- U3 pad 15: /LED_WRNG -> /POT_IN
- U5 pad 5: (no net) -> Net-(C8-Pad1)
- U5 pad 6: (no net) -> /POT_IN
- U5 pad 7: (no net) -> /POT_IN
Routing:
- net /POT_IN: track 0.00 -> 62.8 mm, vias 0 -> 2
- net +3V3: track 158.8 -> 213.2 mm, vias 4 -> 5
- net Net-(C8-Pad1): track 0.00 -> 30.5 mm, vias 0 -> 1
- net GND: track 394.4 -> 419.1 mm
- net /LED_WRNG: track 8.31 -> 0.00 mm
- net /BATT_INPUT: track 32.0 -> 27.2 mm
- net +5V: track 272.4 -> 276.7 mm
- net Net-(D3-Pad2): track 3.05 -> 0.00 mm
- net Net-(D2-Pad1): track 16.0 -> 18.0 mm
Other:
- board text added: "+"
- board text added: "-"
- board text added: "5V to 9V DC INPUT"
- board text added: "HV"

Commit message: PCB Release Candidate
v 0.3
Parts:
- added P15: TP, Pin_Headers:Pin_Header_Straight_1x01, F.Cu at (98.3, 97.0)
- C3: footprint Capacitors_Elko_ThroughHole:Elko_vert_11.2x6.3mm_RM2.5 -> Capacitors_ThroughHole:C_Radial_D10_L20_P2.5-5
- C4: value 4u7 -> 22u; footprint Capacitors_Elko_ThroughHole:Elko_vert_11.2x6.3mm_RM2.5 -> Capacitors_ThroughHole:C_Radial_D10_L20_P2.5-5
- U3: footprint Housings_DIP:DIP-20_W7.62mm_LongPads -> Housings_SSOP:TSSOP-20_4.4x6.5mm_Pitch0.65mm
- U4: value TPS76533 -> LD1117S33CTR; footprint Housings_SOIC:SOIC-8_3.9x4.9mm_Pitch1.27mm -> SOT-223
- moved C5 44.3 mm to (66.6, 126.2), turned to 270 degrees
- moved D2 42.6 mm to (95.0, 123.9)
- moved R8 42.5 mm to (93.6, 127.1)
- moved R15 35.7 mm to (81.2, 117.3), turned to 180 degrees
- moved Q4 31.0 mm to (84.8, 120.3)
- moved RV1 27.5 mm to (127.4, 111.8)
- moved SP1 24.1 mm to (99.1, 116.2)
- moved U5 23.9 mm to (112.1, 114.2)
- moved C8 23.9 mm to (112.4, 119.5)
- moved P10 23.9 mm to (106.2, 111.4)
- moved SW3 15.2 mm to (60.5, 105.2), turned to 90 degrees
- moved P3 12.6 mm to (85.3, 71.8)
- moved SW2 10.2 mm to (60.5, 120.0), turned to 90 degrees
- moved U4 9.35 mm to (78.7, 71.8)
- moved Y1 9.27 mm to (70.4, 117.6)
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Connections:
- U1 pad 1: Net-(U1-Pad1) -> (no net)
- U4 pad 1: Net-(U4-Pad1) -> GND
- U4 pad 2: Net-(U4-Pad2) -> +3V3
- U4 pad 3: GND -> +5V
- U4 pad 4: GND -> (no net)
Routing:
- net +5V: track 276.7 -> 250.6 mm, vias 0 -> 2
- net /PULSE_IN: track 48.9 -> 74.3 mm, vias 3 -> 0
- net GND: track 419.1 -> 396.3 mm, vias 1 -> 2
- net /LCD_LD_B: track 28.2 -> 6.21 mm
- net +3V3: track 213.2 -> 191.2 mm
- net /LCD_LD: track 10.8 -> 28.8 mm, vias 0 -> 2
- net /USER_BTN: track 13.5 -> 31.0 mm, vias 0 -> 2
- net Net-(D2-Pad1): track 18.0 -> 34.3 mm
- net /POT_IN: track 62.8 -> 47.2 mm
- net Net-(C8-Pad1): track 30.5 -> 17.6 mm, vias 1 -> 0
- net /RST: track 17.2 -> 29.2 mm
- net /LCD_D6: track 11.2 -> 22.6 mm, vias 0 -> 1
- net /LCD_D5: track 11.2 -> 22.3 mm, vias 0 -> 1
- net /TEST: track 6.10 -> 16.2 mm
- net +BATT: track 29.6 -> 19.5 mm, vias 2 -> 0
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Other:
- net class Default: clearance 0.3 -> 0.1524
- rule trace_clearance: 0.3 -> 0.1524
- board text added: "+3.3V"
- board text added: "+5V"
- board text added: "A+"
- board text added: "Contador GM Prototipo para Calibración v 0.3"
- board text added: "GM"
- board text added: "HV ADJ"
- board text added: "HV AND DETECTOR"
- board text added: "K-"
- board text added: "ON/OFF SW"
- board text added: "POWER SUPPLY"
- board text added: "RST BTN"
- board text added: "USR BTN"
- board text added: "User Interface & Microcontroller"
- board text removed: "Contador GM"

Commit message: PCB Submission to SeeedStudio
Parts:
- added P16: TP, Measurement_Points:Measurement_Point_Round-TH_Small, F.Cu at (78.3, 63.8)
- DS1: footprint Display:WC1602A -> Socket_Strips:Socket_Strip_Straight_1x16
Other:
- board text added: "1"
- board text added: "16"
